File: riffle-thpr-v0.1.brd (EAGLE design)
At the start: 51.2 x 18 mm, 24 parts, among them U1 BMP180, U2 ADS1115IDGST, U3 TSL2561

Commit message: update
Parts:
- removed SV1: (no value), con-lstb:MA07-1
- added IN4, IN5: 1X2-3.5MM, adafruit:1X2-3.5MM
- added JP3: (no value), SparkFun:1X04-SMD
- moved SJ1 11.3 mm to (46.1, 11.7), turned to 270 degrees
- moved SJ2 5.83 mm to (46.1, 6.40), turned to 90 degrees
Connections:
- net A0: now also JP3.2; no longer SV1.2
- net D3: now also JP3.1; no longer SV1.1
- net GND: now also IN5.2, JP3.4; no longer SV1.7
- net RXD: now also IN4.1; no longer SV1.3
- net TXD: now also IN4.2; no longer SV1.4
- net VBAT: now also JP3.3; no longer SV1.5
- net VCC: now also IN5.1; no longer SV1.6
Routing:
- net D10: track 64.4 -> 16.7 mm, vias 5 -> 0
- net N$5: track 65.8 -> 30.2 mm, vias 1 -> 3
- net SCL: track 68.7 -> 93.2 mm, vias 6 -> 5
- net SDA: track 63.0 -> 79.0 mm, vias 7 -> 4
- net A0: track 55.8 -> 42.4 mm, vias 0 -> 3
- net VCC: track 106.8 -> 120.0 mm, vias 7 -> 3
- net TXD: track 48.7 -> 60.4 mm, vias 2 -> 0
- net MISO: track 22.5 -> 12.0 mm
- net AIN1: track 25.2 -> 16.7 mm, vias 0 -> 2
- net RXD: track 58.5 -> 51.5 mm, vias 1 -> 0
- net AIN3: track 20.5 -> 14.4 mm
- net D3: track 54.8 -> 49.3 mm, vias 1 -> 2
- net N$3: track 5.19 -> 10.5 mm, vias 0 -> 2
- net N$6: track 15.7 -> 20.3 mm
- net MOSI: track 10.8 -> 14.4 mm
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Other:
- board size 51.2 x 18 mm -> 54.4 x 18 mm
