File: riffle-thpr-v0.1.sch (EAGLE design)
At the start: 24 parts, among them U1 BMP180, U2 ADS1115IDGST, U3 TSL2561

Commit message: update
Parts:
- removed SV1: (no value), con-lstb:MA07-1
- added IN4, IN5: 1X2-3.5MM, adafruit:1X2-3.5MM
- added JP3: (no value), SparkFun:M04SMD
Connections:
- net A0: now also JP3.2; no longer SV1.2
- net D3: now also JP3.1; no longer SV1.1
- net GND: now also IN5.2, JP3.4; no longer SV1.7
- net RXD: now also IN4.1; no longer SV1.3
- net TXD: now also IN4.2; no longer SV1.4
- net VBAT: now also JP3.3; no longer SV1.5
- net VCC: now also IN5.1; no longer SV1.6
Changed lines of the file:
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@@
 <layer number="19" name="Unrouted" color="6" fill="1" visible="no" active="no"/>
 <layer number="20" name="Dimension" color="15" fill="1" visible="no" active="no"/>
-<layer number="21" name="tPlace" color="16" fill="1" visible="no" active="no"/>
+<layer number="21" name="tPlace" color="7" fill="1" visible="no" active="no"/>
 <layer number="22" name="bPlace" color="7" fill="1" visible="no" active="no"/>
 <layer number="23" name="tOrigins" color="15" fill="1" visible="no" active="no"/>
@@
 <part name="SUPPLY6" library="supply2" deviceset="GND" device=""/>
 <part name="SUPPLY8" library="supply2" deviceset="GND" device=""/>
-<part name="SV1" library="con-lstb" deviceset="MA07-1" device=""/>
-<part name="P+9" library="SparkFun" deviceset="VCC" device="" value="3.3V"/>
 <part name="C4" library="SparkFun" deviceset="CAP" device="0603-CAP" value="1uF"/>
 <part name="C2" library="SparkFun" deviceset="CAP" device="0603-CAP" value="1uF"/>
@@
 <part name="SUPPLY11" library="supply2" deviceset="GND" device=""/>
 <part name="P+12" library="SparkFun" deviceset="VCC" device="" value="3.3V"/>
+<part name="IN4" library="adafruit" deviceset="1X2" device="-3.5MM"/>
+<part name="IN5" library="adafruit" deviceset="1X2" device="-3.5MM"/>
+<part name="JP3" library="SparkFun" deviceset="M04" device="SMD"/>
+<part name="SUPPLY12" library="supply2" deviceset="GND" device=""/>
+<part name="P+9" library="SparkFun" deviceset="VCC" device="" value="3.3V"/>
+<part name="SUPPLY13" library="supply2" deviceset="GND" device=""/>
 </parts>
 <sheets>
@@
 <instance part="SUPPLY6" gate="GND" x="-194.056" y="16.51"/>
 <instance part="SUPPLY8" gate="GND" x="-203.962" y="16.51"/>
-<instance part="SV1" gate="1" x="17.526" y="65.278" rot="R180"/>
-<instance part="P+9" gate="1" x="-6.604" y="60.198"/>
 <instance part="C4" gate="G$1" x="-141.224" y="121.412" smashed="yes" rot="R180">
 <attribute name="NAME" x="-134.366" y="123.317" size="1.778" layer="95" rot="R180"/>
@@
 <instance part="SUPPLY11" gate="GND" x="-10.16" y="88.9"/>
 <instance part="P+12" gate="1" x="-123.698" y="126.492"/>
+<instance part="IN4" gate="G$1" x="38.1" y="70.866"/>
+<instance part="IN5" gate="G$1" x="39.878" y="60.706"/>
+<instance part="JP3" gate="G$1" x="12.7" y="71.12" rot="R180"/>
+<instance part="SUPPLY12" gate="GND" x="34.798" y="58.166"/>
+<instance part="P+9" gate="1" x="34.798" y="63.246"/>
+<instance part="SUPPLY13" gate="GND" x="7.62" y="63.5"/>
 </instances>
 <busses>
@@
 <pinref part="SUPPLY8" gate="GND" pin="GND"/>
 <wire x1="-203.962" y1="21.082" x2="-203.962" y2="19.05" width="0.1524" layer="91"/>
-</segment>
-<segment>
-<pinref part="SV1" gate="1" pin="7"/>
-<wire x1="9.906" y1="57.658" x2="6.096" y2="57.658" width="0.1524" layer="91"/>
-<label x="2.032" y="57.658" size="1.778" layer="95"/>
 </segment>
 <segment>
@@
 <junction x="-10.16" y="93.98"/>
 <junction x="-10.16" y="91.44"/>
+</segment>
+<segment>
+<pinref part="IN5" gate="G$1" pin="2"/>
+<pinref part="SUPPLY12" gate="GND" pin="GND"/>
+</segment>
+<segment>
+<pinref part="JP3" gate="G$1" pin="4"/>
+<pinref part="SUPPLY13" gate="GND" pin="GND"/>
 </segment>
 </net>
@@
 </segment>
 <segment>
-<pinref part="SV1" gate="1" pin="6"/>
-<pinref part="P+9" gate="1" pin="VCC"/>
-<wire x1="-6.604" y1="60.198" x2="9.906" y2="60.198" width="0.1524" layer="91"/>
-</segment>
-<segment>
 <pinref part="U1" gate="G$1" pin="VDD"/>
 <pinref part="P+10" gate="1" pin="VCC"/>
@@
 <junction x="-123.698" y="126.492"/>
 </segment>
+<segment>
+<pinref part="IN5" gate="G$1" pin="1"/>
+<pinref part="P+9" gate="1" pin="VCC"/>
+</segment>
 </net>
 <net name="N$4" class="0">
@@
 </segment>
 <segment>
-<pinref part="SV1" gate="1" pin="5"/>
-<wire x1="9.906" y1="62.738" x2="6.096" y2="62.738" width="0.1524" layer="91"/>
-<wire x1="6.096" y1="62.738" x2="6.096" y2="62.484" width="0.1524" layer="91"/>
-<label x="1.778" y="62.484" size="1.778" layer="95"/>
+<wire x1="7.62" y1="68.58" x2="1.016" y2="68.58" width="0.1524" layer="91"/>
+<wire x1="1.016" y1="68.58" x2="1.016" y2="68.326" width="0.1524" layer="91"/>
+<label x="-3.556" y="67.818" size="1.778" layer="95"/>
+<pinref part="JP3" gate="G$1" pin="3"/>
 </segment>
 </net>
@@
 </segment>
 <segment>
-<pinref part="SV1" gate="1" pin="2"/>
-<wire x1="9.906" y1="70.358" x2="5.588" y2="70.358" width="0.1524" layer="91"/>
-<label x="3.302" y="70.612" size="1.778" layer="95"/>
+<wire x1="7.62" y1="71.12" x2="0.762" y2="71.12" width="0.1524" layer="91"/>
+<label x="-1.524" y="71.374" size="1.778" layer="95"/>
+<pinref part="JP3" gate="G$1" pin="2"/>
 </segment>
 </net>
@@
 </segment>
 <segment>
-<pinref part="SV1" gate="1" pin="1"/>
-<wire x1="9.906" y1="72.898" x2="5.334" y2="72.898" width="0.1524" layer="91"/>
-<label x="3.302" y="73.152" size="1.778" layer="95"/>
+<wire x1="7.62" y1="73.66" x2="0.508" y2="73.66" width="0.1524" layer="91"/>
+<label x="-1.524" y="73.914" size="1.778" layer="95"/>
+<pinref part="JP3" gate="G$1" pin="1"/>
 </segment>
 </net>
@@
 </segment>
 <segment>
-<pinref part="SV1" gate="1" pin="3"/>
-<wire x1="9.906" y1="67.818" x2="5.588" y2="67.818" width="0.1524" layer="91"/>
-<label x="3.048" y="68.072" size="1.778" layer="95"/>
+<pinref part="IN4" gate="G$1" pin="1"/>
+<wire x1="33.02" y1="73.406" x2="27.94" y2="73.406" width="0.1524" layer="91"/>
+<label x="24.13" y="73.406" size="1.778" layer="95"/>
 </segment>
 </net>
@@
 </segment>
 <segment>
-<pinref part="SV1" gate="1" pin="4"/>
-<wire x1="9.906" y1="65.278" x2="5.588" y2="65.278" width="0.1524" layer="91"/>
-<label x="2.286" y="65.532" size="1.778" layer="95"/>
-</segment>
-</net>
+<pinref part="IN4" gate="G$1" pin="2"/>
+<wire x1="33.02" y1="70.866" x2="28.194" y2="70.866" width="0.1524" layer="91"/>
+<label x="23.622" y="70.866" size="1.778" layer="95"/>
+</segment>
+</net>
